Commit message: update

File: ros_urdf/urdf/ur5e_onsga.urdf (robot description, URDF)
Before this commit: robot mobile_manipulator, 15 links, 14 joints
Links:
- link onrobotsg_base_link: geometry collision mesh filename=package://onrobotsg_description/meshes/collision/plate_and_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 scale=0.001 0.001 0.001; visual mesh filename=package://onrobotsg_description/meshes/visual/sga_full.STL scale=0.001 0.001 0.001
